File: pcb/ADXL345_Accelerometer/ADXL345_Accelerometer.kicad_pcb (KiCad board)
At the start: 2 copper layers, 25.4 x 22.9 mm, 16 parts, among them J1 Conn_01x09, Q1 BSS138, Q2 BSS138, U1 ADXL345_Library, U2 AP2112K-3.3

Commit message: Correcciones
Se corrigieron de acuerdo a las recomendaciones realizadas por el alumno revisor.
Parts:
- moved D1 0.52 mm to (141.0, 96.5)
- moved R5 0.32 mm to (153.6, 96.4)
Routing:
- net GND: track 14.5 -> 17.3 mm
- net /SDO\ADDR: track 45.3 -> 44.7 mm
- net /SCL: vias 0 -> 2
