File: pcb/ADXL345_Accelerometer/ADXL345_Accelerometer.kicad_pcb (KiCad board)
At the start: 2 copper layers, 25.4 x 22.9 mm, 18 parts, among them J1 Conn_01x09, Q1 BSS138, Q2 BSS138, U1 ADXL345BCCZ, U2 AP2112K-3.3

Commit message: Correccciones
Other:
- board text added: "Grilla: 0,1270 mm/5.00 mils Vias: 0.9/0.5mm Pistas: 0.25mm, 0.5mm Margen: 0.40 mm Terminación: HASL"
- board text removed: "Grilla: 0,1 mm Ancho de las pistas: 0,25 mm Vias: 0.9/0.5mm Pistas: 0.25mm, 0.5mm Margen: 0.40 mm Terminación: HASL"
